File: v1.2/alarm_panel.kicad_sch (KiCad schematic)
At the start: 85 parts, among them J1 Screw_Terminal_01x03, J10 Barrel_Jack, J11 Conn_01x03_Female, J12 Conn_01x04_Male, J13 Conn_02x07_Odd_Even, J14 Conn_02x10_Odd_Even, J15 Conn_02x10_Odd_Even, J2 Screw_Terminal_01x03, J3 Screw_Terminal_01x03, J4 Screw_Terminal_01x03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

Commit message: Add files via upload
Parts:
- U6: footprint QuinLED-ESP32-KiCad6:QuinLED-ESP32 -> alarm_panel:QuinLED-ESP32
Connections:
- net 3V3: now also J12.2 (Pin_2); no longer J12.1 (Pin_1)
- net GND: now also J12.1 (Pin_1); no longer J12.2 (Pin_2)
Changed lines of the file:
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@@
     (stroke (width 0) (type default) (color 0 0 0 0))
   )
-  (wire (pts (xy 156.6164 70.2564) (xy 165.6588 70.2564))
+  (wire (pts (xy 156.6164 67.7164) (xy 165.6588 67.7164))
     (stroke (width 0) (type default) (color 0 0 0 0))
   )
@@
     )
   )
-  (global_label "3V3" (shape input) (at 156.6164 67.7164 0) (fields_autoplaced)
+  (global_label "3V3" (shape input) (at 156.6164 70.2564 0) (fields_autoplaced)
     (effects (font (size 1.27 1.27)) (justify left))
-    (property "Intersheet References" "${INTERSHEET_REFS}" (id 0) (at 163.1419 67.7958 0)
+    (property "Intersheet References" "${INTERSHEET_REFS}" (id 0) (at 163.1419 70.3358 0)
       (effects (font (size 1.27 1.27)) (justify left) hide)
     )
@@
       (effects (font (size 1.27 1.27)) (justify left))
     )
-    (property "Footprint" "QuinLED-ESP32-KiCad6:QuinLED-ESP32" (id 2) (at 165.1 20.066 0)
+    (property "Footprint" "alarm_panel:QuinLED-ESP32" (id 2) (at 165.1 20.066 0)
       (effects (font (size 1.27 1.27)) hide)
     )
@@
     (pin "2")
   )
-  (symbol (lib_id "power:GND") (at 165.6588 70.2564 0) (unit 1)
+  (symbol (lib_id "power:GND") (at 165.6588 67.7164 0) (unit 1)
     (in_bom yes) (on_board yes) (fields_autoplaced)
-    (property "Reference" "#PWR08" (id 0) (at 165.6588 76.6064 0)
+    (property "Reference" "#PWR08" (id 0) (at 165.6588 74.0664 0)
       (effects (font (size 1.27 1.27)) hide)
     )
-    (property "Value" "GND" (id 1) (at 165.6588 74.8284 0))
-    (property "Footprint" "" (id 2) (at 165.6588 70.2564 0)
+    (property "Value" "GND" (id 1) (at 165.6588 72.2884 0))
+    (property "Footprint" "" (id 2) (at 165.6588 67.7164 0)
       (effects (font (size 1.27 1.27)) hide)
     )
-    (property "Datasheet" "" (id 3) (at 165.6588 70.2564 0)
+    (property "Datasheet" "" (id 3) (at 165.6588 67.7164 0)
       (effects (font (size 1.27 1.27)) hide)
     )
@@
     )
     (path "/425d4a83-d0e9-45a7-9f4f-eceebc4f2de8"
-      (reference "U6") (unit 1) (value "QuinLED-ESP32") (footprint "QuinLED-ESP32-KiCad6:QuinLED-ESP32")
+      (reference "U6") (unit 1) (value "QuinLED-ESP32") (footprint "alarm_panel:QuinLED-ESP32")
     )
   )
